Commit message: Refactor URDF and launch files to support namespaced Gazebo topics and improve simulation configuration

File: nav2_minimal_tb4_description/urdf/icreate/common_properties.urdf.xacro (robot description, xacro)
@@ -44,5 +44,5 @@
     params="sensor_name gazebo update_rate visualize
             h_samples h_res h_min_angle h_max_angle
-            r_min r_max r_res *plugin">
+            r_min r_max r_res namespace:='' *plugin">
     <sensor name="${sensor_name}" type="gpu_lidar">
       <update_rate>${update_rate}</update_rate>
@@ -50,5 +50,5 @@
       <always_on>true</always_on>
       <gz_frame_id>${sensor_name}_link</gz_frame_id>
-      <topic>scan</topic>
+      <topic>${namespace}/scan</topic>
       <lidar>
         <scan>

File: nav2_minimal_tb4_description/urdf/icreate/create3.urdf.xacro (robot description, xacro)
@@ -94,7 +94,7 @@
         <max_angular_velocity>2.0</max_angular_velocity>
         <min_angular_velocity>-2.0</min_angular_velocity>
-        <topic>/cmd_vel</topic>
-        <odom_topic>/odom</odom_topic>
-        <tf_topic>tf</tf_topic>
+        <topic>$(arg namespace)/cmd_vel</topic>
+        <odom_topic>$(arg namespace)/odom</odom_topic>
+        <tf_topic>$(arg namespace)/tf</tf_topic>
         <frame_id>odom</frame_id>
         <child_frame_id>base_link</child_frame_id>
@@ -106,5 +106,5 @@
         <joint_name>left_wheel_joint</joint_name>
         <joint_name>right_wheel_joint</joint_name>
-        <topic>joint_states</topic>
+        <topic>$(arg namespace)/joint_states</topic>
         <update_rate>30</update_rate>
       </plugin>

File: nav2_minimal_tb4_description/urdf/icreate/sensors/imu.urdf.xacro (robot description, xacro)
@@ -14,5 +14,5 @@
       <always_on>true</always_on>
       <update_rate>${update_rate}</update_rate>
-      <topic>imu</topic>
+      <topic>${namespace}/imu</topic>
       <imu>
         <angular_velocity>

File: nav2_minimal_tb4_description/urdf/sensors/oakd.urdf.xacro (robot description, xacro)
@@ -1,5 +1,5 @@
 <?xml version="1.0"?>
 <robot xmlns:xacro="http://ros.org/wiki/xacro">
-<xacro:macro name="oakd" params="name:=oakd parent_link *origin model:=pro">
+<xacro:macro name="oakd" params="name:=oakd parent_link *origin model:=pro namespace:=''">
   <xacro:include filename="$(find nav2_minimal_tb4_description)/urdf/icreate/common_properties.urdf.xacro"/>
   <xacro:property name="mass"       value="0.061"/>
@@ -115,5 +115,5 @@
       <update_rate>10</update_rate>
       <visualize>true</visualize>
-      <topic>rgbd_camera</topic>
+      <topic>${namespace}/rgbd_camera</topic>
     </sensor>
     <xacro:material_darkgray/>

File: nav2_minimal_tb4_description/urdf/sensors/rplidar.urdf.xacro (robot description, xacro)
@@ -1,5 +1,5 @@
 <?xml version="1.0"?>
 <robot xmlns:xacro="http://ros.org/wiki/xacro">
-<xacro:macro name="rplidar" params="name parent_link gazebo *origin">
+<xacro:macro name="rplidar" params="name parent_link gazebo namespace:='' *origin">
   <xacro:include filename="$(find nav2_minimal_tb4_description)/urdf/icreate/common_properties.urdf.xacro"/>
   <xacro:property name="mass"       value="0.17"/>
@@ -33,5 +33,5 @@
                   update_rate="10.0" visualize="true"
                   h_samples="360" h_res="1.0" h_min_angle="0.000" h_max_angle="6.280000"
-                  r_min="0.164" r_max="20.0" r_res="0.01">
+                  r_min="0.164" r_max="20.0" r_res="0.01" namespace="${namespace}">
                   <plugin name="dummy" filename="dummyfile"></plugin>
     </xacro:ray_sensor>

File: nav2_minimal_tb4_description/urdf/standard/turtlebot4.urdf.xacro (robot description, xacro)
@@ -1,4 +1,6 @@
 <?xml version="1.0" ?>
 <robot name="turtlebot4" xmlns:xacro="http://ros.org/wiki/xacro">
+  <!-- Namespace for Gazebo topics -->
+  <xacro:arg name="namespace" default=""/>
   <!-- Base create3 model -->
   <xacro:include filename="$(find nav2_minimal_tb4_description)/urdf/icreate/create3.urdf.xacro" />
@@ -110,5 +112,5 @@
   </xacro:tower_sensor_plate>
   <!-- Turtlebot4 sensor definitions -->
-  <xacro:rplidar name="rplidar" parent_link="shell_link" gazebo="$(arg gazebo)">
+  <xacro:rplidar name="rplidar" parent_link="shell_link" gazebo="$(arg gazebo)" namespace="$(arg namespace)">
     <origin xyz="${rplidar_x_offset} ${rplidar_y_offset} ${rplidar_z_offset}"
             rpy="0 0 ${pi/2}"/>
@@ -117,5 +119,5 @@
     <origin xyz="${camera_mount_x_offset} ${camera_mount_y_offset} ${camera_mount_z_offset}"/>
   </xacro:camera_bracket>
-  <xacro:oakd model="pro" parent_link="oakd_camera_bracket">
+  <xacro:oakd model="pro" parent_link="oakd_camera_bracket" namespace="$(arg namespace)">
     <origin xyz="${oakd_pro_x_offset} ${oakd_pro_y_offset} ${oakd_pro_z_offset}"/>
   </xacro:oakd>
