Commit message: Update URDF and launch files for faster and simpler simulation

File: nav2_minimal_tb4_description/urdf/icreate/bumper.urdf.xacro (robot description, xacro)
@@ -24,15 +24,23 @@
   <link name="${link_name}">
     <visual>
+      <origin xyz="0.08 0 0" rpy="0 0 0"/>
       <geometry>
-        <mesh filename="${visual_mesh}"/>
+        <box size="0.20 0.25 0.08"/>
       </geometry>
+      <material name="darkgrey">
+        <color rgba="0.2 0.2 0.2 1"/>
+      </material>
     </visual>
     <collision>
+      <origin xyz="0.08 0 0.05" rpy="0 0 0"/>
       <geometry>
-        <mesh filename="${collision_mesh}"/>
+        <box size="0.20 0.25 0.08"/>
       </geometry>
     </collision>
     <xacro:insert_block name="inertial"/>
   </link>
+  <gazebo reference="${link_name}">
+    <material>Gazebo/DarkGrey</material>
+  </gazebo>
   <xacro:dummy_bumper_zone
       name="bump_front_center">

File: nav2_minimal_tb4_description/urdf/icreate/create3.urdf.xacro (robot description, xacro)
@@ -12,5 +12,6 @@
   <!-- Mechanical properties -->
   <xacro:property name="body_z_offset"           value="${-2.5*cm2m}" />
-  <xacro:property name="body_collision_z_offset" value="${1*cm2m}" />
+  <!-- Raise collision up to avoid floor penetration when spawning (more clearance) -->
+  <xacro:property name="body_collision_z_offset" value="${3*cm2m}" />
   <xacro:property name="body_mass"               value="2.300" />
   <xacro:property name="body_radius"             value="${16.4*cm2m}" />
@@ -31,11 +32,14 @@
   <link name="base_link">
     <visual>
-      <origin xyz="0 0 ${body_z_offset + base_link_z_offset}" rpy="0 0 ${pi/2}"/>
+      <origin xyz="0 0 ${body_z_offset + base_link_z_offset}" rpy="0 0 0"/>
       <geometry>
-        <mesh filename="package://nav2_minimal_tb4_description/meshes/body_visual.dae" />
+        <cylinder length="${body_length}" radius="${body_radius}"/>
       </geometry>
+      <material name="darkgrey">
+        <color rgba="0.3 0.3 0.3 1"/>
+      </material>
     </visual>
     <collision name="create3_base_collision">
-      <origin xyz="0 0 ${body_z_offset + body_collision_z_offset  + base_link_z_offset}" rpy="0 0 ${pi/2}"/>
+      <origin xyz="0 0 ${body_z_offset + body_collision_z_offset  + base_link_z_offset}" rpy="0 0 0"/>
       <geometry>
         <cylinder length="${body_length}" radius="${body_radius}"/>

File: nav2_minimal_tb4_description/urdf/icreate/wheel.urdf.xacro (robot description, xacro)
@@ -30,9 +30,11 @@
   </link>
   <gazebo reference="${wheel_link_name}">
-    <mu1>1.0</mu1>
-    <mu2>1.0</mu2>
-    <kp>1000000.0</kp>
-    <kd>100.0</kd>
-    <minDepth>0.0001</minDepth>
+    <mu1>0.9</mu1>
+    <mu2>0.9</mu2>
+    <slip1>0.1</slip1>
+    <slip2>0.1</slip2>
+    <kp>200000.0</kp>
+    <kd>20.0</kd>
+    <minDepth>0.003</minDepth>
     <maxVel>1.0</maxVel>
     <material>Gazebo/DarkGrey</material>

File: nav2_minimal_tb4_description/urdf/sensors/oakd.urdf.xacro (robot description, xacro)
@@ -21,7 +21,11 @@
   <link name="${base_frame}">
     <visual>
+      <origin xyz="${collision_offset_x} ${collision_offset_y} ${collision_offset_z}" rpy="0 0 0"/>
       <geometry>
-        <mesh filename="package://nav2_minimal_tb4_description/meshes/${name}_${model}.dae" scale="1 1 1" />
+        <box size="${collision_length_x} ${collision_length_y} ${collision_length_z}"/>
       </geometry>
+      <material name="darkgrey">
+        <color rgba="0.15 0.15 0.15 1"/>
+      </material>
     </visual>
     <collision>
@@ -37,4 +41,7 @@
     </inertial>
   </link>
+  <gazebo reference="${base_frame}">
+    <material>Gazebo/DarkGrey</material>
+  </gazebo>
   <!-- RGB Camera -->
   <link name="${name}_rgb_camera_frame">
@@ -114,5 +121,5 @@
       </camera>
       <update_rate>10</update_rate>
-      <visualize>true</visualize>
+      <visualize>false</visualize>
       <topic>${namespace}/rgbd_camera</topic>
     </sensor>

File: nav2_minimal_tb4_description/urdf/sensors/rplidar.urdf.xacro (robot description, xacro)
@@ -31,5 +31,5 @@
   <gazebo reference="${name}_link">
     <xacro:ray_sensor sensor_name="${name}" gazebo="${gazebo}"
-                  update_rate="10.0" visualize="true"
+                  update_rate="10.0" visualize="false"
                   h_samples="360" h_res="1.0" h_min_angle="0.000" h_max_angle="6.280000"
                   r_min="0.164" r_max="20.0" r_res="0.01" namespace="${namespace}">

File: nav2_minimal_tb4_description/urdf/standard/turtlebot4.urdf.xacro (robot description, xacro)
@@ -63,12 +63,16 @@
   <link name="shell_link">
     <visual>
-      <origin xyz="0 0 0" rpy="${pi/2} 0 ${pi/2}"/>
+      <origin xyz="0 0 0" rpy="0 0 0"/>
       <geometry>
-        <mesh filename="package://nav2_minimal_tb4_description/meshes/shell.dae" scale="1 1 1" />
+        <box size="${shell_length} ${shell_radius*2} 0.08"/>
       </geometry>
+      <material name="darkgrey">
+        <color rgba="0.2 0.2 0.2 1"/>
+      </material>
     </visual>
     <collision name="shell_collision">
+      <origin xyz="0 0 0" rpy="0 0 0"/>
       <geometry>
-        <mesh filename="package://nav2_minimal_tb4_description/meshes/shell_collision.dae" scale="1 1 1" />
+        <box size="${shell_length} ${shell_radius*2} 0.08"/>
       </geometry>
     </collision>

Commit message: Improve model. Slighly mroe distance for poximity to offset low temporal resolution, visual improvements

File: nav2_minimal_tb4_description/urdf/icreate/bumper.urdf.xacro (robot description, xacro)
@@ -24,7 +24,7 @@
   <link name="${link_name}">
     <visual>
-      <origin xyz="0.08 0 0" rpy="0 0 0"/>
+      <origin xyz="0.015 0 0" rpy="0 0 0"/>
       <geometry>
-        <box size="0.20 0.25 0.08"/>
+        <cylinder radius="0.17" length="0.03"/>
       </geometry>
       <material name="darkgrey">
@@ -33,7 +33,7 @@
     </visual>
     <collision>
-      <origin xyz="0.08 0 0.05" rpy="0 0 0"/>
+      <origin xyz="0.015 0 0" rpy="0 0 0"/>
       <geometry>
-        <box size="0.20 0.25 0.08"/>
+        <cylinder radius="0.164" length="0.03"/>
       </geometry>
     </collision>

File: nav2_minimal_tb4_description/urdf/icreate/wheel.urdf.xacro (robot description, xacro)
@@ -36,5 +36,5 @@
     <kp>200000.0</kp>
     <kd>20.0</kd>
-    <minDepth>0.003</minDepth>
+    <minDepth>0.001</minDepth>
     <maxVel>1.0</maxVel>
     <material>Gazebo/DarkGrey</material>

File: nav2_minimal_tb4_description/urdf/sensors/proximity.urdf.xacro (robot description, xacro)
@@ -19,5 +19,5 @@
         </geometry>
         <material name="proximity_sensor_black">
-          <color rgba="0.1 0.1 0.1 1"/>
+          <color rgba="0.0 0.0 0.0 1"/>
         </material>
       </visual>
@@ -33,5 +33,5 @@
       <sensor name="${name}" type="gpu_lidar">
         <always_on>true</always_on>
-        <update_rate>5</update_rate>
+        <update_rate>6</update_rate>
         <visualize>false</visualize>
         <topic>${namespace}/proximity/${name}</topic>
@@ -48,10 +48,10 @@
           <range>
             <min>0.01</min>
-            <max>0.10</max>
+            <max>0.15</max>
             <resolution>0.01</resolution>
           </range>
         </lidar>
       </sensor>
-      <material>Gazebo/DarkGrey</material>
+      <material>Gazebo/Black</material>
     </gazebo>
   </xacro:macro>

File: nav2_minimal_tb4_description/urdf/standard/turtlebot4.urdf.xacro (robot description, xacro)
@@ -132,5 +132,5 @@
   </xacro:oakd>
   <!-- Proximity sensors ring on base_link -->
-  <xacro:proximity_ring parent_link="base_link" gazebo="$(arg gazebo)" namespace="$(arg namespace)" radius="0.16" z_offset="0.12"/>
+  <xacro:proximity_ring parent_link="base_link" gazebo="$(arg gazebo)" namespace="$(arg namespace)" radius="0.16" z_offset="0.05"/>
   <!-- Ground truth odometry publisher for Gazebo -->
   <xacro:arg name="gazebo" default=""/>
