Commit message: create toggle for lidar, fix global clock

File: nav2_minimal_tb4_description/urdf/standard/turtlebot4.urdf.xacro (robot description, xacro)
@@ -3,4 +3,6 @@
   <!-- Namespace for Gazebo topics -->
   <xacro:arg name="namespace" default=""/>
+  <!-- Enable/disable RPLIDAR sensor (set to 0 to disable for performance testing) -->
+  <xacro:property name="enable_rplidar" value="0" />
   <!-- Base create3 model -->
   <xacro:include filename="$(find nav2_minimal_tb4_description)/urdf/icreate/create3.urdf.xacro" />
@@ -117,8 +119,10 @@
   </xacro:tower_sensor_plate>
   <!-- Turtlebot4 sensor definitions -->
-  <xacro:rplidar name="rplidar" parent_link="shell_link" gazebo="$(arg gazebo)" namespace="$(arg namespace)">
-    <origin xyz="${rplidar_x_offset} ${rplidar_y_offset} ${rplidar_z_offset}"
-            rpy="0 0 ${pi/2}"/>
-  </xacro:rplidar>
+  <xacro:if value="${enable_rplidar}">
+    <xacro:rplidar name="rplidar" parent_link="shell_link" gazebo="$(arg gazebo)" namespace="$(arg namespace)">
+      <origin xyz="${rplidar_x_offset} ${rplidar_y_offset} ${rplidar_z_offset}"
+              rpy="0 0 ${pi/2}"/>
+    </xacro:rplidar>
+  </xacro:if>
   <xacro:camera_bracket name="oakd_camera_bracket">
     <origin xyz="${camera_mount_x_offset} ${camera_mount_y_offset} ${camera_mount_z_offset}"/>
